File: TempFilter.kicad_sch (KiCad schematic)
At the start: 4 parts

Commit message: board done
Parts:
- C1: p/n (none) -> CC0805JRX7R9BB473
- R1: p/n (none) -> RT0805FRE074K7L
- R2: p/n (none) -> RT0805FRE0710KL
