File: TempFilter.kicad_sch (KiCad schematic)
At the start: 4 parts

Commit message: shrug
Parts:
- C1: LCSC Part # (none) -> C1745
- R1: LCSC Part # (none) -> C17673
- R2: LCSC Part # (none) -> C17414
Changed lines of the file:
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@@
+					(unit 1)
+				)
+				(path "/0e9575a4-1ede-4f13-af58-a4e2eef0ca4e/b5b39d26-996d-4b80-8b0b-95fc6ddade53"
+					(reference "#PWR07")
 					(unit 1)
 				)
@@
 			)
 		)
+		(property "LCSC Part #" "C1745"
+			(at 133.985 105.41 90)
+			(effects
+				(font
+					(size 1.27 1.27)
+				)
+				(hide yes)
+			)
+		)
+		(property "JLC-p/n" ""
+			(at 133.985 105.41 0)
+			(effects
+				(font
+					(size 1.27 1.27)
+				)
+			)
+		)
 		(pin "1"
 		)
@@
 				(path "/0e9575a4-1ede-4f13-af58-a4e2eef0ca4e/aefbee89-cedd-4224-8d34-e19c3f8712a6"
 					(reference "C8")
+					(unit 1)
+				)
+				(path "/0e9575a4-1ede-4f13-af58-a4e2eef0ca4e/b5b39d26-996d-4b80-8b0b-95fc6ddade53"
+					(reference "C17")
 					(unit 1)
 				)
@@
 			)
 		)
+		(property "LCSC Part #" "C17673"
+			(at 142.24 100.33 90)
+			(effects
+				(font
+					(size 1.27 1.27)
+				)
+				(hide yes)
+			)
+		)
+		(property "JLC-p/n" ""
+			(at 142.24 100.33 0)
+			(effects
+				(font
+					(size 1.27 1.27)
+				)
+			)
+		)
 		(pin "1"
 		)
@@
 				(path "/0e9575a4-1ede-4f13-af58-a4e2eef0ca4e/aefbee89-cedd-4224-8d34-e19c3f8712a6"
 					(reference "R15")
+					(unit 1)
+				)
+				(path "/0e9575a4-1ede-4f13-af58-a4e2eef0ca4e/b5b39d26-996d-4b80-8b0b-95fc6ddade53"
+					(reference "R34")
 					(unit 1)
 				)
@@
 					(unit 1)
 				)
+				(path "/0e9575a4-1ede-4f13-af58-a4e2eef0ca4e/b5b39d26-996d-4b80-8b0b-95fc6ddade53"
+					(reference "#PWR09")
+					(unit 1)
+				)
 				(path "/0e9575a4-1ede-4f13-af58-a4e2eef0ca4e/bc64ba2a-0992-412a-9240-778b52a7b51f"
 					(reference "#PWR060")
@@
 			)
 		)
+		(property "LCSC Part #" "C17414"
+			(at 147.955 92.71 90)
+			(effects
+				(font
+					(size 1.27 1.27)
+				)
+				(hide yes)
+			)
+		)
+		(property "JLC-p/n" ""
+			(at 147.955 92.71 0)
+			(effects
+				(font
+					(size 1.27 1.27)
+				)
+			)
+		)
 		(pin "1"
 		)
@@
 				(path "/0e9575a4-1ede-4f13-af58-a4e2eef0ca4e/aefbee89-cedd-4224-8d34-e19c3f8712a6"
 					(reference "R16")
+					(unit 1)
+				)
+				(path "/0e9575a4-1ede-4f13-af58-a4e2eef0ca4e/b5b39d26-996d-4b80-8b0b-95fc6ddade53"
+					(reference "R35")
 					(unit 1)
 				)
@@
 			)
 		)
+		(property "JLC-p/n" ""
+			(at 132.08 97.79 0)
+			(effects
+				(font
+					(size 1.27 1.27)
+				)
+			)
+		)
 		(pin "1"
 		)
@@
 					(unit 1)
 				)
+				(path "/0e9575a4-1ede-4f13-af58-a4e2eef0ca4e/b5b39d26-996d-4b80-8b0b-95fc6ddade53"
+					(reference "TP19")
+					(unit 1)
+				)
